File: MC_Series/channel.kicad_sch (KiCad schematic)
At the start: 15 parts, among them J1 Screw_Terminal_01x02, K1 Channel 1, Q1 2N3904, SW1 SW_Slide_DPDT, U1 PC817, U2 H11AA1

Commit message: Updated MC_Series template
Parts:
- removed J1: Screw_Terminal_01x02, nelees:1017503, symbol Connector:Screw_Terminal_01x02
- added CH_OUT1: Screw_Terminal_01x02, symbol Connector:Screw_Terminal_01x02
- added C_RC_FILTER1: 100nF, symbol Device:C
- added C_SNUB1: 100nF, symbol Device:C_Polarized
- added D_ESD_F_RA1, D_ESD_F_SP1: ESD5Z3.3, Diode_SMD:D_SOD-523, symbol Diode:ESD5Zxx
- added F_CH1: Littelfuse 273.200, symbol Device:Fuse
- added MOV_CH_PROTECT1: S14K275, symbol Device:Varistor
- added R_RELAY_PULLUP1: 10k, symbol Device:R
- added R_SNUB1: 100, symbol Device:R
- added T_3V1, T_GND1: T_3V3, symbol Connector:TestPoint
- added T_F_RA_1: T_F_RA, symbol Connector:TestPoint
- added T_F_SP_1: T_F_SP, symbol Connector:TestPoint
- added T_RC1: T_RC, symbol Connector:TestPoint
- CH_RELAY1: renamed from K1; value Channel 1 -> Channel
- R_HI_LIMIT1: renamed from R6; value 10k -> 1k
- R_OPTO_PWR1: renamed from R1; value 1k -> 4.7k
- renumbered C1 to C_FRA_FILTER1, D1 to D_RELAY_FLYBACK1, U2 to OPTO_RA_FEEDBACK1, U1 to OPTO_RC_CTRL1, Q1 to Q_RELAY_DRV1, SW1 to RELAY_MODE_SEL1, R2 to R_DRV_BASE1, R7 to R_FRA_PULLUP1, R5 to R_LOW_LIMIT1, R3 to R_OPTO_RA_AC1_1, R4 to R_OPTO_RA_AC2_1
Connections:
- net AC_L: now also C_SNUB1.1, MOV_CH_PROTECT1.1
- net AC_N: now also CH_OUT1.1 (Pin_1)
- net F_RA: now also D_ESD_F_RA1.1 (K), T_F_RA_1.1
- net F_SP: now also RELAY_MODE_SEL1.5 (B), D_ESD_F_SP1.1 (K), T_F_SP_1.1; no longer R_LOW_LIMIT1.1
- net GND: now also R_LOW_LIMIT1.1, C_RC_FILTER1.2, D_ESD_F_RA1.2 (A), D_ESD_F_SP1.2 (A), T_GND1.1; no longer RELAY_MODE_SEL1.4 (A)
- net RC: now also C_RC_FILTER1.1, R_RELAY_PULLUP1.1, T_RC1.1
- net at OPTO_RA_FEEDBACK1.1: now also R_OPTO_RA_AC2_1.2; no longer R_OPTO_RA_AC2_1.1
- net at R_OPTO_RA_AC1_1.1: now also R_OPTO_RA_AC2_1.1; no longer RELAY_MODE_SEL1.2 (B)
- net at R_OPTO_RA_AC1_1.2: now also RELAY_MODE_SEL1.2 (B), F_CH1.2, MOV_CH_PROTECT1.2, R_SNUB1.2; no longer R_OPTO_RA_AC2_1.2
- net at RELAY_MODE_SEL1.6 (C): now also R_HI_LIMIT1.1; no longer R_HI_LIMIT1.2
- net at R_LOW_LIMIT1.2: now also RELAY_MODE_SEL1.4 (A); no longer RELAY_MODE_SEL1.5 (B)
- net +3V3 renamed 3V3
- net 3V3: now also R_HI_LIMIT1.2, T_3V1.1; no longer R_HI_LIMIT1.1
- net +5V renamed 5V0
- net 5V0: now also R_RELAY_PULLUP1.2
- new net: CH_OUT1.2 (Pin_2), F_CH1.1
- new net: C_SNUB1.2, R_SNUB1.1
- no-connect marks 0 -> 1
Other:
- title: (none) -> Channel
- moved on the sheet: C_FRA_FILTER1, D_RELAY_FLYBACK1, OPTO_RA_FEEDBACK1, OPTO_RC_CTRL1, Q_RELAY_DRV1, RELAY_MODE_SEL1, R_FRA_PULLUP1
